File: PCBs/Interfaceboard/Measurements.sch (KiCad schematic (older format))
At the start: 9 parts

Commit message: Added most circuits from Interface schematic provided by Rakesh. Lacks a few connectors, transistors, and optocouplers. Needs connections for Zybo. Awaiting feedback from meeting with Rakesh.
Parts:
- added C? (x4): 10n, symbol Device:C
- added C? (x5): 100n, symbol Device:C
- added C? (x2): 1u, symbol Device:C
- added C?: 10u, symbol Device:C
- added D?: BAV16W, Diode_SMD:D_SOD-123, symbol Diode:BAV16W
- added R? (x5): 3.3k, symbol Device:R
- added R? (x3): 33k, symbol Device:R
- added R? (x2): 4.7k, symbol Device:R
- added R?: 680, symbol Device:R
- added R?: 100k, symbol Device:R
- added R? (x8): 10k, symbol Device:R
- added R? (x2): 150k, symbol Device:R
- added R? (x4): NM, symbol Device:R
- added R?: 6.8k, symbol Device:R
- added R? (x2): 2.2k, symbol Device:R
- added R?: 0, symbol Device:R
- added R?: 1k, symbol Device:R
- added R? (x2): 22k, symbol Device:R
- added U?: AD8603, Package_TO_SOT_SMD:TSOT-23-5, symbol Amplifier_Operational:AD8603
- added U? (x3): MCP6L02x-xSN, Package_SO:SOIC-8_3.9x4.9mm_P1.27mm, symbol Amplifier_Operational:MCP6L02x-xSN
- added U?: ACPL-C870, Package_SO:SSO-8_6.8x5.9mm_P1.27mm_Clearance8mm, symbol Isolator_Analog:ACPL-C870
- added U? (x3): AD8606ARMZ-REEL, ElectricGoKart:AD8606ARMZ-REEL, symbol ElectricGoKart:AD8606ARMZ-REEL
Connections:
- net labels added: +5V, +5V_Batt, +BATT, BattVolt_Meas, Drive_Switch_Supp, Foot_Switch_Supp, GND, GND_Batt, Motor_Therm_Raw, Overtemp_Meas
- net labels removed: Drive_Switch, Foot_Switch
- wire segments 23 -> 197
- no-connect marks 0 -> 1
Other:
- note added: "ADC Input Protection"
- note added: "Active low digital signal to Zybo"
- note added: "High motor temperature detection"
- note added: "Isolated battery voltage measurement"
- note added: "Power and parked op amp\nIf AD8606 is not placed in close vicinity:\nAdd 1-10 µF decoupling capacitor."
- note added: "TORQUE"
- note added: "Trigger point:\n1.284 V ~~143 C\nHysteresis ~~19 C"
- note removed: "high motor temperature detection wip"
- note removed: "op amp"
