File: PCBs/Interfaceboard/PWM.sch (KiCad schematic (older format))
At the start: 0 parts

Commit message: Added most circuits from Interface schematic provided by Rakesh. Lacks a few connectors, transistors, and optocouplers. Needs connections for Zybo. Awaiting feedback from meeting with Rakesh.
Parts:
- added C? (x2): 1u, symbol Device:C
- added R? (x12): 100, symbol Device:R
- added U?: Si8660AB-B-IS1, ElectricGoKart:Si8660AB-B-IS1, symbol ElectricGoKart:Si8660AB-B-IS1
Connections:
- net labels added: +3V3, +5V_Float, GND, GND_Float, PWM1_A, PWM1_B, PWM2_A, PWM2_B, PWM3_A, PWM3_B, Zybo_PWM1_A, Zybo_PWM1_B, Zybo_PWM2_A, Zybo_PWM2_B, Zybo_PWM3_A, Zybo_PWM3_B
- wire segments 0 -> 36
Other:
- note added: "Isolated gate driver signals"
