File: PCBs/Interfaceboard/Power.sch (KiCad schematic (older format))
At the start: 0 parts

Commit message: Added most circuits from Interface schematic provided by Rakesh. Lacks a few connectors, transistors, and optocouplers. Needs connections for Zybo. Awaiting feedback from meeting with Rakesh.
Parts:
- added C? (x2): 100u, symbol Device:C
- added C? (x11): 1u, symbol Device:C
- added C? (x4): 1n, symbol Device:C
- added C? (x2): 10n, symbol Device:C
- added R? (x2): NM, symbol Device:R
- added U?: TEN20-4823WIN, Converter_DCDC:Converter_DCDC_TRACO_TEN20-xxxx_THT, symbol Converter_DCDC:TEN20-4823WIN
- added U?: TVN 5-4811WI, ElectricGoKart:TVN_5_4811WI, symbol ElectricGoKart:TVN_5-4811WI
- added U?: LP2985-5.0, Package_TO_SOT_SMD:SOT-23-5, symbol Regulator_Linear:LP2985-5.0
- added U?: LP2985-3.3, Package_TO_SOT_SMD:SOT-23-5, symbol Regulator_Linear:LP2985-3.3
Connections:
- net labels added: +15V, +3V3_Ref, +5V, +5V_Ref, +BATT, -15V, GND, GND_Batt
- wire segments 0 -> 103
- no-connect marks 0 -> 2
Other:
- note added: "3.3 V reference voltage"
- note added: "5 V reference voltage"
- note added: "Auxiliary supplies needed"
- note added: "Isolated +-15V DC-DC Converter"
- note added: "Isolated 5 V DC-DC Converter"
