File: PCBs/Interfaceboard/RelayControl.sch (KiCad schematic (older format))
At the start: 0 parts

Commit message: Added most circuits from Interface schematic provided by Rakesh. Lacks a few connectors, transistors, and optocouplers. Needs connections for Zybo. Awaiting feedback from meeting with Rakesh.
Parts:
- added D?: 1N4148W, Diode_SMD:D_SOD-123, symbol Diode:1N4148W
- added Q?: BC856, Package_TO_SOT_SMD:SOT-23, symbol Transistor_BJT:BC856
- added R? (x2): 1k, symbol Device:R
- added R?: 33k, symbol Device:R
- added R?: 100k, symbol Device:R
- added R? (x8): 20, symbol Device:R
- added R? (x2): 47k, symbol Device:R
- added R?: 10k, symbol Device:R
Connections:
- net labels added: +3V3, +BATT, Base, GND, GND_Batt, PreCharge_En, Precharge_Out, Relay_En, Relay_In, Relay_Out
- wire segments 0 -> 45
Other:
- note added: "4 x 20R (2512)"
- note added: "Main relay control circuit"
- note added: "Precharge circuit"
- note added: "optocoupler"
- note added: "transistor"
