File: PCBs/Interfaceboard/Connectors.sch (KiCad schematic (older format))
At the start: 10 parts, among them J301 TSW-105-07-T-D, J302 TSW-105-07-T-D, J304 TSW-105-07-T-D, J305 TSW-105-07-T-D

Commit message: Removed some buttons and added LEDs. Finished placing the components on the PCB.
Changed lines of the file:
@@
 Wire Wire Line
 	4200 1900 4250 1900
-Text HLabel 4200 3000 0    50   BiDi ~ 0
+Text HLabel 4200 3000 0    50   Input ~ 0
 Digital1
 Wire Wire Line
 	4200 3000 4250 3000
-Text HLabel 4200 3100 0    50   BiDi ~ 0
+Text HLabel 4200 3100 0    50   Output ~ 0
 Digital2
 Wire Wire Line
 	4200 3100 4250 3100
-Text HLabel 4200 3200 0    50   BiDi ~ 0
+Text HLabel 4200 3200 0    50   Output ~ 0
 Digital3
 Wire Wire Line
 	4200 3200 4250 3200
-Text HLabel 4200 3300 0    50   BiDi ~ 0
+Text HLabel 4200 3300 0    50   Output ~ 0
 Digital4
 Wire Wire Line
 	4200 3300 4250 3300
-Text HLabel 4200 3400 0    50   BiDi ~ 0
+Text HLabel 4200 3400 0    50   Output ~ 0
 Digital5
 Wire Wire Line

Commit message: Changed M2 to M3 hole. Vias are free.
Parts:
- H1, H2: value M2 Mount -> M3 Mount; footprint MountingHole:MountingHole_2.1mm -> MountingHole:MountingHole_3.2mm_M3
Changed lines of the file:
@@
 P 3900 4200
 F 0 "H1" H 4000 4246 50  0000 L CNN
-F 1 "M2 Mount" H 4000 4155 50  0000 L CNN
-F 2 "MountingHole:MountingHole_2.1mm" H 3900 4200 50  0001 C CNN
+F 1 "M3 Mount" H 4000 4155 50  0000 L CNN
+F 2 "MountingHole:MountingHole_3.2mm_M3" H 3900 4200 50  0001 C CNN
 F 3 "~" H 3900 4200 50  0001 C CNN
 	1    3900 4200
@@
 P 4700 4200
 F 0 "H2" H 4800 4246 50  0000 L CNN
-F 1 "M2 Mount" H 4800 4155 50  0000 L CNN
-F 2 "MountingHole:MountingHole_2.1mm" H 4700 4200 50  0001 C CNN
+F 1 "M3 Mount" H 4800 4155 50  0000 L CNN
+F 2 "MountingHole:MountingHole_3.2mm_M3" H 4700 4200 50  0001 C CNN
 F 3 "~" H 4700 4200 50  0001 C CNN
 	1    4700 4200
