File: PCBs/Interfaceboard/Torque.sch (KiCad schematic (older format))
At the start: 0 parts

Commit message: Removed interface board, added analog interface board.
Other:
- note removed: "CONTAINS SIGNALS TO/FROM ZYBO"
Changed lines of the file:
@@
 $Descr A4 11693 8268
 encoding utf-8
-Sheet 9 9
+Sheet 1 4
 Title "Interface Board for Control of PMAC Motor in Electric Go-Kart"
-Date "2021-02-23"
+Date "2021-03-04"
 Rev "Version 1"
 Comp "University of Southern Denmark"
@@
 Comment4 ""
 $EndDescr
-Text Notes 4350 3900 0    100  ~ 0
-CONTAINS SIGNALS TO/FROM ZYBO
 $EndSCHEMATC

Commit message: Finished schematics for analog interface board. Ready for review and then PCB design.
Parts:
- added C14: 10µ, Capacitor_SMD:C_0805_2012Metric, symbol Device:C
- added C15: 100n, Capacitor_SMD:C_0603_1608Metric, symbol Device:C
- added C16: 30n, Capacitor_SMD:C_0603_1608Metric, symbol Device:C
- added C17: 33n, Capacitor_SMD:C_0603_1608Metric, symbol Device:C
- added C18: 56n, Capacitor_SMD:C_0603_1608Metric, symbol Device:C
- added D3: 2.5 V, Diode_SMD:D_SOD-523, symbol Device:D_Zener_Small
- added R15: 9.88k, Resistor_SMD:R_0603_1608Metric, symbol Device:R
- added R16, R17: 7.5k, Resistor_SMD:R_0603_1608Metric, symbol Device:R
- added R18: 147, Resistor_SMD:R_0603_1608Metric, symbol Device:R
- added R19: 10k, Resistor_SMD:R_0603_1608Metric, symbol Device:R
- added U3: MCP6L01x-xOT, Package_TO_SOT_SMD:SOT-23-5, symbol Amplifier_Operational:MCP6L01x-xOT
Connections:
- net labels added: +3V3_Ref, +5V, GND, Torque_ADC, Torque_Pedal
- wire segments 0 -> 37
Other:
- note added: "R_pot = 0 Ohm to 7.5 kOhm\n\nTorque output:\n3.3 V * (R_pot || R_L) / (R_pot || R_L + R_H) = 0 V to 1 V"
- note added: "Sallen-Key cutoff:\n517 Hz\n\nRC cutoff:\n1/(2*pi*147*33*10^-9) = 32.8 kHz"
- note added: "Torque pedal measurement"

Commit message: Added test points and final associated footprints. Made outline for PCB.
Parts:
- added TP3: TestPoint, TestPoint:TestPoint_Plated_Hole_D2.0mm, symbol Connector:TestPoint
- D3: value 2.5 V -> 3.3 V; Name ESD5Z2.5T5G -> ESD5Z3.3T1G
Connections:
- wire segments 37 -> 38
Changed lines of the file:
@@
 $Descr A4 11693 8268
 encoding utf-8
-Sheet 3 4
-Title "Interface Board for Control of PMAC Motor in Electric Go-Kart"
-Date "2021-03-04"
+Sheet 3 5
+Title "Analog Board for Control of PMAC Motor in Electric Go-Kart"
+Date "2021-03-13"
 Rev "Version 1"
 Comp "University of Southern Denmark"
@@
 P 1900 2000
 F 0 "D3" V 1854 2070 50  0000 L CNN
-F 1 "2.5 V" V 1945 2070 50  0000 L CNN
+F 1 "3.3 V" V 1945 2070 50  0000 L CNN
 F 2 "Diode_SMD:D_SOD-523" V 1900 2000 50  0001 C CNN
 F 3 "https://www.mouser.dk/datasheet/2/308/ESD5Z2_5T1_D-1522641.pdf" V 1900 2000 50  0001 C CNN
-F 4 "ESD5Z2.5T5G" V 1900 2000 50  0001 C CNN "Name"
+F 4 "ESD5Z3.3T1G" V 1900 2000 50  0001 C CNN "Name"
 	1    1900 2000
 	0    1    1    0
@@
 Text Notes 900  3450 0    50   ~ 0
 R_pot = 0 Ohm to 7.5 kOhm\n\nTorque output:\n3.3 V * (R_pot || R_L) / (R_pot || R_L + R_H) = 0 V to 1 V
+$Comp
+L Connector:TestPoint TP?
+U 1 1 604E435E
+P 4500 1700
+AR Path="/6040B450/604E435E" Ref="TP?"  Part="1"
+AR Path="/6040B46E/604E435E" Ref="TP3"  Part="1"
+F 0 "TP3" H 4550 1850 50  0000 L CNN
+F 1 "TestPoint" H 4550 1750 50  0001 L CNN
+F 2 "TestPoint:TestPoint_Plated_Hole_D2.0mm" H 4700 1700 50  0001 C CNN
+F 3 "~" H 4700 1700 50  0001 C CNN
+	1    4500 1700
+	1    0    0    -1
+$EndComp
+Wire Wire Line
+	4500 1700 4500 1850
 $EndSCHEMATC

Commit message: Made changes to resistor sizes and footprints. Placed switches on PCB, ready for the rest.
Parts:
- R15: value 9.88k -> 11.5k
Other:
- note added: "R_pot = 0 Ohm to 7.5 kOhm\n\nTorque output:\n3.3 V * (R_pot || R_L) / (R_pot || R_L + R_H) = 0 V to 0.9 V\n\n> 0.9 V means pedal disconnected."
- note removed: "R_pot = 0 Ohm to 7.5 kOhm\n\nTorque output:\n3.3 V * (R_pot || R_L) / (R_pot || R_L + R_H) = 0 V to 1 V"
Changed lines of the file:
@@
 P 1700 1500
 F 0 "R15" H 1750 1500 50  0000 L CNN
-F 1 "9.88k" V 1700 1400 50  0000 L CNN
+F 1 "11.5k" V 1700 1400 50  0000 L CNN
 F 2 "Resistor_SMD:R_0603_1608Metric" V 1630 1500 50  0001 C CNN
 F 3 "~" H 1700 1500 50  0001 C CNN
@@
 Wire Wire Line
 	1900 2100 1900 2200
-Text Notes 900  3450 0    50   ~ 0
-R_pot = 0 Ohm to 7.5 kOhm\n\nTorque output:\n3.3 V * (R_pot || R_L) / (R_pot || R_L + R_H) = 0 V to 1 V
+Text Notes 900  3550 0    50   ~ 0
+R_pot = 0 Ohm to 7.5 kOhm\n\nTorque output:\n3.3 V * (R_pot || R_L) / (R_pot || R_L + R_H) = 0 V to 0.9 V\n\n> 0.9 V means pedal disconnected.
 $Comp
 L Connector:TestPoint TP?

Commit message: Minor changes to schematics, removed test points, placed a few components on PCB.
Parts:
- removed TP3: TestPoint, TestPoint:TestPoint_Plated_Hole_D2.0mm, symbol Connector:TestPoint
Connections:
- wire segments 38 -> 37
Changed lines of the file:
@@
 Text Notes 900  3550 0    50   ~ 0
 R_pot = 0 Ohm to 7.5 kOhm\n\nTorque output:\n3.3 V * (R_pot || R_L) / (R_pot || R_L + R_H) = 0 V to 0.9 V\n\n> 0.9 V means pedal disconnected.
-$Comp
-L Connector:TestPoint TP?
-U 1 1 604E435E
-P 4500 1700
-AR Path="/6040B450/604E435E" Ref="TP?"  Part="1"
-AR Path="/6040B46E/604E435E" Ref="TP3"  Part="1"
-F 0 "TP3" H 4550 1850 50  0000 L CNN
-F 1 "TestPoint" H 4550 1750 50  0001 L CNN
-F 2 "TestPoint:TestPoint_Plated_Hole_D2.0mm" H 4700 1700 50  0001 C CNN
-F 3 "~" H 4700 1700 50  0001 C CNN
-	1    4500 1700
-	1    0    0    -1
-$EndComp
-Wire Wire Line
-	4500 1700 4500 1850
 $EndSCHEMATC
