File: PCBs/Interfaceboard/Torque.sch (KiCad schematic (older format))
At the start: 0 parts

Commit message: Merge of 'Analog Board' into main (#2)
* Added analog board schematics and finished PCB.
* Added a few documentation files.
Parts:
- added C14: 10µ, Capacitor_SMD:C_0805_2012Metric, symbol Device:C
- added C15: 100n, Capacitor_SMD:C_0603_1608Metric, symbol Device:C
- added C16: 30n, Capacitor_SMD:C_0603_1608Metric, symbol Device:C
- added C17: 33n, Capacitor_SMD:C_0603_1608Metric, symbol Device:C
- added C18: 56n, Capacitor_SMD:C_0603_1608Metric, symbol Device:C
- added D3: 3.3 V, Diode_SMD:D_SOD-523, symbol Device:D_Zener_Small
- added R15: 11.5k, Resistor_SMD:R_0603_1608Metric, symbol Device:R
- added R16, R17: 7.5k, Resistor_SMD:R_0603_1608Metric, symbol Device:R
- added R18: 147, Resistor_SMD:R_0603_1608Metric, symbol Device:R
- added R19: 10k, Resistor_SMD:R_0603_1608Metric, symbol Device:R
- added U3: MCP6L01x-xOT, Package_TO_SOT_SMD:SOT-23-5, symbol Amplifier_Operational:MCP6L01x-xOT
Connections:
- net labels added: +3V3_Ref, +5V, GND, Torque_ADC, Torque_Pedal
- wire segments 0 -> 37
Other:
- note added: "R_pot = 0 Ohm to 7.5 kOhm\n\nTorque output:\n3.3 V * (R_pot || R_L) / (R_pot || R_L + R_H) = 0 V to 0.9 V\n\n> 0.9 V means pedal disconnected."
- note added: "Sallen-Key cutoff:\n517 Hz\n\nRC cutoff:\n1/(2*pi*147*33*10^-9) = 32.8 kHz"
- note added: "Torque pedal measurement"
