File: PCBs/Interfaceboard/Currents.sch (KiCad schematic (older format))
At the start: 0 parts

Commit message: Removed interface board, added analog interface board.
Other:
- note removed: "CONTAINS USB ISOLATOR TO BE CONNECTED TO ZYBO"
Changed lines of the file:
@@
 $Descr A4 11693 8268
 encoding utf-8
-Sheet 8 9
+Sheet 1 4
 Title "Interface Board for Control of PMAC Motor in Electric Go-Kart"
-Date "2021-02-23"
+Date "2021-03-04"
 Rev "Version 1"
 Comp "University of Southern Denmark"
@@
 Comment4 ""
 $EndDescr
-Text Notes 3400 3900 0    100  ~ 0
-CONTAINS USB ISOLATOR TO BE CONNECTED TO ZYBO
 $EndSCHEMATC

Commit message: Added analog board hierarchial sheets. Started work on connectors, supply, and in amp for phase current measurements.
Parts:
- added C? (x2): 100n, symbol Device:C
- added C? (x2): 10µ, symbol Device:C
- added C?: 1n, symbol Device:C
- added C? (x2): 100p, symbol Device:C
- added D?: D_TVS, symbol Device:D_TVS
- added FB? (x2): <50 mA, 600R, symbol Device:Ferrite_Bead_Small
- added R?: 28.8, symbol Device:R
- added R?: 3.2, symbol Device:R
- added R? (x2): R, symbol Device:R
- added R? (x2): 20k, symbol Device:R
- added U?: AD8420ARMZ, ElectricGoKart:AD8420ARMZ, symbol ElectricGoKart:AD8420ARMZ
Connections:
- net labels added: +15V, +15V_Filt, +3V3_Ref, +5V_Ref, -15V, -15V_Filt, 0V5, GND, Phase1_ADC, Phase1_In, Phase2_ADC, Phase2_In
- wire segments 0 -> 56
Other:
- note added: "Choose one"
- note added: "Offset voltage"
- note added: "P = 0.08 W"
- note added: "P = 0.7 W"
- note added: "Power supply stabilization"
- note added: "RFI Filter:\nf_c,diff = 1/(2*pi*R*(2*C_common+C_ground)) = 3789 Hz\nf_c,comm = 1/(2*pi*R*C_ground) = 79577 Hz\n\nDifferential phase delay at 333 Hz:\n-arctan(2*pi*333*R*(2*C_common+C_ground)) = -5 degrees"

Commit message: Finished schematics for analog interface board. Ready for review and then PCB design.
Parts:
- removed FB?: <50 mA, 600R, symbol Device:Ferrite_Bead_Small
- added C10, C12, C6: 100n, Capacitor_SMD:C_0603_1608Metric, symbol Device:C
- added C7, C9: 100p, Capacitor_SMD:C_0603_1608Metric, symbol Device:C
- added C8: 1n, Capacitor_SMD:C_0603_1608Metric, symbol Device:C
- added D2: 5 V, Diode_SMD:D_SOD-523, symbol Device:D_TVS
- added FB2: 400 mA, 1k5, Inductor_SMD:L_0805_2012Metric, symbol Device:Ferrite_Bead_Small
- added R10, R2, R8: sot, symbol Device:R
- added R11, R12, R5: sot, Resistor_SMD:R_0603_1608Metric, symbol Device:R
- added R7, R9: 20k, Resistor_SMD:R_0603_1608Metric, symbol Device:R
- added U2: AD8420ARMZ, ElectricGoKart:AD8420ARMZ, symbol ElectricGoKart:AD8420ARMZ
- C1, C2, C3, C4, C5: renamed from C?; footprint (none) -> Capacitor_SMD:C_0603_1608Metric
- C11, C13: renamed from C?; footprint (none) -> Capacitor_SMD:C_0805_2012Metric
- D1: renamed from D?; value D_TVS -> 5 V; footprint (none) -> Diode_SMD:D_SOD-523; Name (none) -> DESD5V0U1BB-7
- FB1: renamed from FB?; value <50 mA, 600R -> 400 mA, 1k5; footprint (none) -> Inductor_SMD:L_0805_2012Metric; Name (none) -> HZ0805D152R-10
- R1, R3: renamed from R?; footprint (none) -> Resistor_SMD:R_0603_1608Metric
- R13: renamed from R?; value R -> 5.6k; footprint (none) -> Resistor_SMD:R_0603_1608Metric
- R14: renamed from R?; value R -> 1k; footprint (none) -> Resistor_SMD:R_0603_1608Metric
- R4: renamed from R?; value 28.8 -> sot
- R6: renamed from R?; value 3.2 -> sot; footprint (none) -> Resistor_SMD:R_0603_1608Metric
- gave numbers to parts that had none: 1
Connections:
- net labels removed: +5V_Ref
- wire segments 56 -> 131
Other:
- note added: "3.3 V * 1000/(5600+1000) = 0.5 V"
- note added: "Caps 5%"
- note added: "Phase 1 current measurement"
- note added: "Phase 2 current measurement"
- note added: "Tolerance <1%"
- note added: "sot"
- note removed: "Choose one"

Commit message: Added test points and final associated footprints. Made outline for PCB.
Parts:
- added TP1, TP2: TestPoint, TestPoint:TestPoint_Plated_Hole_D2.0mm, symbol Connector:TestPoint
- R10, R2, R4, R8: footprint (none) -> Resistor_SMD:R_1206_3216Metric
Connections:
- wire segments 131 -> 135

Commit message: Made changes to resistor sizes and footprints. Placed switches on PCB, ready for the rest.
Parts:
- R10, R4: value sot -> 56; footprint Resistor_SMD:R_1206_3216Metric -> Resistor_SMD:R_1210_3225Metric; Name (none) -> RC1210FR-0756RL
- R11, R5: value sot -> 3.09; Name (none) -> CRCW06033R09FKEA
- R12, R6: value sot -> DNP
- R2, R8: value sot -> 54.9; footprint Resistor_SMD:R_1206_3216Metric -> Resistor_SMD:R_1210_3225Metric; Name (none) -> ERJ-14NF54R9U
Other:
- note added: "P = 0.73 W"
- note added: "Tolerance =<1%"
- note removed: "P = 0.7 W"
Changed lines of the file:
@@
 P 2150 1750
 F 0 "R4" V 2250 1750 50  0000 C CNN
-F 1 "sot" V 2150 1750 50  0000 C CNN
-F 2 "Resistor_SMD:R_1206_3216Metric" V 2080 1750 50  0001 C CNN
-F 3 "~" H 2150 1750 50  0001 C CNN
+F 1 "56" V 2150 1750 50  0000 C CNN
+F 2 "Resistor_SMD:R_1210_3225Metric" V 2080 1750 50  0001 C CNN
+F 3 "https://www.mouser.dk/datasheet/2/447/PYu_RC_Group_51_RoHS_L_10-1664068.pdf" H 2150 1750 50  0001 C CNN
+F 4 "RC1210FR-0756RL" V 2150 1750 50  0001 C CNN "Name"
 	1    2150 1750
 	0    1    1    0
@@
 P 2650 1950
 F 0 "R6" H 2600 1950 50  0000 R CNN
-F 1 "sot" V 2650 2000 50  0000 R CNN
+F 1 "DNP" V 2650 2050 50  0000 R CNN
 F 2 "Resistor_SMD:R_0603_1608Metric" V 2580 1950 50  0001 C CNN
 F 3 "~" H 2650 1950 50  0001 C CNN
@@
 P 2550 1950
 F 0 "R5" H 2700 1950 50  0000 R CNN
-F 1 "sot" V 2550 2000 50  0000 R CNN
+F 1 "3.09" V 2550 2050 50  0000 R CNN
 F 2 "Resistor_SMD:R_0603_1608Metric" V 2480 1950 50  0001 C CNN
-F 3 "~" H 2550 1950 50  0001 C CNN
+F 3 "https://www.mouser.dk/datasheet/2/427/dcrcwe3-1762152.pdf" H 2550 1950 50  0001 C CNN
+F 4 "CRCW06033R09FKEA" H 2550 1950 50  0001 C CNN "Name"
 	1    2550 1950
 	-1   0    0    1
@@
 P 2150 1650
 F 0 "R2" V 2050 1650 50  0000 C CNN
-F 1 "sot" V 2150 1650 50  0000 C CNN
-F 2 "Resistor_SMD:R_1206_3216Metric" V 2080 1650 50  0001 C CNN
-F 3 "~" H 2150 1650 50  0001 C CNN
+F 1 "54.9" V 2150 1650 50  0000 C CNN
+F 2 "Resistor_SMD:R_1210_3225Metric" V 2080 1650 50  0001 C CNN
+F 3 "https://www.mouser.dk/datasheet/2/315/AOA0000C304-1149620.pdf" H 2150 1650 50  0001 C CNN
+F 4 "ERJ-14NF54R9U" V 2150 1650 50  0001 C CNN "Name"
 	1    2150 1650
 	0    1    1    0
@@
 	4800 1550 4950 1550
 Connection ~ 4800 1550
-Text Notes 1950 1500 0    50   ~ 0
-P = 0.7 W
+Text Notes 1900 1500 0    50   ~ 0
+P = 0.73 W
 Wire Wire Line
 	2550 1700 2650 1700
@@
 Wire Notes Line
 	2800 4850 2800 5700
-$Comp
-L Device:R R10
-U 1 1 604B0FAD
-P 2150 3800
-F 0 "R10" V 2250 3800 50  0000 C CNN
-F 1 "sot" V 2150 3800 50  0000 C CNN
-F 2 "Resistor_SMD:R_1206_3216Metric" V 2080 3800 50  0001 C CNN
-F 3 "~" H 2150 3800 50  0001 C CNN
-	1    2150 3800
-	0    1    1    0
-$EndComp
-$Comp
-L Device:R R12
-U 1 1 604B0FB9
-P 2650 4000
-F 0 "R12" H 2600 4000 50  0000 R CNN
-F 1 "sot" V 2650 4050 50  0000 R CNN
-F 2 "Resistor_SMD:R_0603_1608Metric" V 2580 4000 50  0001 C CNN
-F 3 "~" H 2650 4000 50  0001 C CNN
-	1    2650 4000
-	-1   0    0    1
-$EndComp
 $Comp
 L power:GND #PWR0108
@@
 Text Notes 2400 4200 0    50   ~ 0
 P = 0.08 W
-$Comp
-L Device:R R11
-U 1 1 604B102B
-P 2550 4000
-F 0 "R11" H 2750 4000 50  0000 R CNN
-F 1 "sot" V 2550 4050 50  0000 R CNN
-F 2 "Resistor_SMD:R_0603_1608Metric" V 2480 4000 50  0001 C CNN
-F 3 "~" H 2550 4000 50  0001 C CNN
-	1    2550 4000
-	-1   0    0    1
-$EndComp
-$Comp
-L Device:R R8
-U 1 1 604B1031
-P 2150 3700
-F 0 "R8" V 2050 3700 50  0000 C CNN
-F 1 "sot" V 2150 3700 50  0000 C CNN
-F 2 "Resistor_SMD:R_1206_3216Metric" V 2080 3700 50  0001 C CNN
-F 3 "~" H 2150 3700 50  0001 C CNN
-	1    2150 3700
-	0    1    1    0
-$EndComp
 Wire Wire Line
 	2550 4150 2550 4250
@@
 	4800 3600 4950 3600
 Connection ~ 4800 3600
-Text Notes 1950 3550 0    50   ~ 0
-P = 0.7 W
+Text Notes 1900 3550 0    50   ~ 0
+P = 0.73 W
 Wire Wire Line
 	2550 3750 2650 3750
@@
 Text Notes 2900 1600 0    50   ~ 0
 Caps 5%
-Text Notes 1850 2300 0    50   ~ 0
-Tolerance <1%
+Text Notes 1800 2300 0    50   ~ 0
+Tolerance =<1%
 Text Notes 2900 3650 0    50   ~ 0
 Caps 5%
-Text Notes 1850 4350 0    50   ~ 0
-Tolerance <1%
+Text Notes 1800 4350 0    50   ~ 0
+Tolerance =<1%
 Text Notes 3450 4950 0    50   ~ 0
 Tolerance <1%
@@
 	5000 1550 4950 1550
 Connection ~ 4950 1550
+$Comp
+L Device:R R11
+U 1 1 604E9E51
+P 2550 4000
+F 0 "R11" H 2700 4000 50  0000 R CNN
+F 1 "3.09" V 2550 4100 50  0000 R CNN
+F 2 "Resistor_SMD:R_0603_1608Metric" V 2480 4000 50  0001 C CNN
+F 3 "https://www.mouser.dk/datasheet/2/427/dcrcwe3-1762152.pdf" H 2550 4000 50  0001 C CNN
+F 4 "CRCW06033R09FKEA" H 2550 4000 50  0001 C CNN "Name"
+	1    2550 4000
+	-1   0    0    1
+$EndComp
+$Comp
+L Device:R R12
+U 1 1 604EA7D1
+P 2650 4000
+F 0 "R12" H 2600 4000 50  0000 R CNN
+F 1 "DNP" V 2650 4100 50  0000 R CNN
+F 2 "Resistor_SMD:R_0603_1608Metric" V 2580 4000 50  0001 C CNN
+F 3 "~" H 2650 4000 50  0001 C CNN
+	1    2650 4000
+	-1   0    0    1
+$EndComp
+$Comp
+L Device:R R10
+U 1 1 604F4513
+P 2150 3800
+F 0 "R10" V 2250 3800 50  0000 C CNN
+F 1 "56" V 2150 3800 50  0000 C CNN
+F 2 "Resistor_SMD:R_1210_3225Metric" V 2080 3800 50  0001 C CNN
+F 3 "https://www.mouser.dk/datasheet/2/447/PYu_RC_Group_51_RoHS_L_10-1664068.pdf" H 2150 3800 50  0001 C CNN
+F 4 "RC1210FR-0756RL" V 2150 3800 50  0001 C CNN "Name"
+	1    2150 3800
+	0    1    1    0
+$EndComp
+$Comp
+L Device:R R8
+U 1 1 604F451A
+P 2150 3700
+F 0 "R8" V 2050 3700 50  0000 C CNN
+F 1 "54.9" V 2150 3700 50  0000 C CNN
+F 2 "Resistor_SMD:R_1210_3225Metric" V 2080 3700 50  0001 C CNN
+F 3 "https://www.mouser.dk/datasheet/2/315/AOA0000C304-1149620.pdf" H 2150 3700 50  0001 C CNN
+F 4 "ERJ-14NF54R9U" V 2150 3700 50  0001 C CNN "Name"
+	1    2150 3700
+	0    1    1    0
+$EndComp
 $EndSCHEMATC

Commit message: Minor changes to schematics, removed test points, placed a few components on PCB.
Parts:
- removed C12: 100n, Capacitor_SMD:C_0603_1608Metric, symbol Device:C
- removed TP1, TP2: TestPoint, TestPoint:TestPoint_Plated_Hole_D2.0mm, symbol Connector:TestPoint
- added D4: LM4041CFTA, ElectricGoKart:LM4041, symbol ElectricGoKart:LM4041CFTA
- added R20: 1k, Resistor_SMD:R_0603_1608Metric, symbol Device:R
- R13: value 5.6k -> 5.1k
- R14: value 1k -> 1.43k
Connections:
- wire segments 135 -> 129
Other:
- note added: "1.225 V * 1000/(1450+1000) = 0.5 V"
- note added: "1.225 V reference"
- note removed: "3.3 V * 1000/(5600+1000) = 0.5 V"
- note removed: "Tolerance <1%"
- note removed: "sot"
Changed lines of the file:
@@
 	-1   0    0    1
 $EndComp
-$Comp
-L ElectricGoKart:+3V3_Ref #PWR0106
-U 1 1 60491C07
-P 3050 5100
-F 0 "#PWR0106" H 3050 4950 50  0001 C CNN
-F 1 "+3V3_Ref" H 2850 5250 50  0000 L CNN
-F 2 "" H 3050 5100 50  0001 C CNN
-F 3 "" H 3050 5100 50  0001 C CNN
-	1    3050 5100
-	1    0    0    -1
-$EndComp
-$Comp
-L Device:R R13
-U 1 1 60492701
-P 3450 5100
-F 0 "R13" V 3350 5100 50  0000 C CNN
-F 1 "5.6k" V 3450 5100 50  0000 C CNN
-F 2 "Resistor_SMD:R_0603_1608Metric" V 3380 5100 50  0001 C CNN
-F 3 "~" H 3450 5100 50  0001 C CNN
-	1    3450 5100
-	0    1    1    0
-$EndComp
-$Comp
-L Device:R R14
-U 1 1 60492EE9
-P 4050 5100
-F 0 "R14" V 3950 5100 50  0000 C CNN
-F 1 "1k" V 4050 5100 50  0000 C CNN
-F 2 "Resistor_SMD:R_0603_1608Metric" V 3980 5100 50  0001 C CNN
-F 3 "~" H 4050 5100 50  0001 C CNN
-	1    4050 5100
-	0    1    1    0
-$EndComp
-Wire Wire Line
-	3600 5100 3750 5100
-$Comp
-L power:GND #PWR0107
-U 1 1 604933C2
-P 4250 5500
-F 0 "#PWR0107" H 4250 5250 50  0001 C CNN
-F 1 "GND" H 4250 5350 50  0000 C CNN
-F 2 "" H 4250 5500 50  0001 C CNN
-F 3 "" H 4250 5500 50  0001 C CNN
-	1    4250 5500
-	1    0    0    -1
-$EndComp
-Wire Wire Line
-	4200 5100 4250 5100
-Text Label 3700 5100 0    50   ~ 0
-0V5
 Text Label 4300 2000 1    50   ~ 0
 0V5
@@
 Wire Wire Line
 	4800 1550 4700 1550
-Wire Notes Line
-	2800 4850 4400 4850
-Text Notes 2800 5800 0    50   ~ 0
-Offset voltage
 Wire Wire Line
 	4400 1850 4400 2000
@@
 Wire Wire Line
 	2550 2200 2650 2200
-Wire Wire Line
-	4800 1550 4950 1550
 Connection ~ 4800 1550
 Text Notes 1900 1500 0    50   ~ 0
@@
 Wire Wire Line
 	1550 1700 1750 1700
-$Comp
-L Device:C C12
-U 1 1 6049BC99
-P 3750 5300
-F 0 "C12" H 3865 5346 50  0000 L CNN
-F 1 "100n" H 3865 5255 50  0000 L CNN
-F 2 "Capacitor_SMD:C_0603_1608Metric" H 3788 5150 50  0001 C CNN
-F 3 "~" H 3750 5300 50  0001 C CNN
-	1    3750 5300
-	1    0    0    -1
-$EndComp
-Connection ~ 3750 5100
-Wire Wire Line
-	3750 5100 3900 5100
-Wire Wire Line
-	3750 5100 3750 5150
-Text Notes 3500 5350 0    50   ~ 0
-sot
-Wire Wire Line
-	4250 5100 4250 5500
-Wire Wire Line
-	3750 5450 3750 5500
-Wire Wire Line
-	3750 5500 4250 5500
-Connection ~ 4250 5500
-Wire Notes Line
-	4400 5700 2800 5700
-Wire Notes Line
-	2800 4850 2800 5700
 $Comp
 L power:GND #PWR0108
@@
 Wire Wire Line
 	2550 4250 2650 4250
-Wire Wire Line
-	4800 3600 4950 3600
 Connection ~ 4800 3600
 Text Notes 1900 3550 0    50   ~ 0
@@
 Text Notes 1000 4700 0    50   ~ 0
 Phase 2 current measurement
-Wire Wire Line
-	3050 5100 3300 5100
-Wire Notes Line
-	4400 5700 4400 4850
-Text Notes 2800 5950 0    50   ~ 0
-3.3 V * 1000/(5600+1000) = 0.5 V
 Wire Wire Line
 	2100 4950 2100 5050
@@
 Text Notes 1800 4350 0    50   ~ 0
 Tolerance =<1%
-Text Notes 3450 4950 0    50   ~ 0
-Tolerance <1%
-$Comp
-L Connector:TestPoint TP2
-U 1 1 604BAD99
-P 4950 3450
-F 0 "TP2" H 5000 3600 50  0000 L CNN
-F 1 "TestPoint" H 5000 3500 50  0001 L CNN
-F 2 "TestPoint:TestPoint_Plated_Hole_D2.0mm" H 5150 3450 50  0001 C CNN
-F 3 "~" H 5150 3450 50  0001 C CNN
-	1    4950 3450
-	1    0    0    -1
-$EndComp
-Wire Wire Line
-	4950 3450 4950 3600
-Wire Wire Line
-	4950 3600 5000 3600
-Connection ~ 4950 3600
-$Comp
-L Connector:TestPoint TP1
-U 1 1 604C69A1
-P 4950 1400
-F 0 "TP1" H 5000 1550 50  0000 L CNN
-F 1 "TestPoint" H 5000 1450 50  0001 L CNN
-F 2 "TestPoint:TestPoint_Plated_Hole_D2.0mm" H 5150 1400 50  0001 C CNN
-F 3 "~" H 5150 1400 50  0001 C CNN
-	1    4950 1400
-	1    0    0    -1
-$EndComp
-Wire Wire Line
-	4950 1400 4950 1550
-Wire Wire Line
-	5000 1550 4950 1550
-Connection ~ 4950 1550
 $Comp
 L Device:R R11
@@
 	0    1    1    0
 $EndComp
+$Comp
+L ElectricGoKart:+3V3_Ref #PWR07
+U 1 1 604FDECB
+P 3100 5100
+F 0 "#PWR07" H 3100 4950 50  0001 C CNN
+F 1 "+3V3_Ref" H 2900 5250 50  0000 L CNN
+F 2 "" H 3100 5100 50  0001 C CNN
+F 3 "" H 3100 5100 50  0001 C CNN
+	1    3100 5100
+	1    0    0    -1
+$EndComp
+$Comp
+L Device:R R13
+U 1 1 604FDED1
+P 3450 5100
+F 0 "R13" V 3350 5100 50  0000 C CNN
+F 1 "5.1k" V 3450 5100 50  0000 C CNN
+F 2 "Resistor_SMD:R_0603_1608Metric" V 3380 5100 50  0001 C CNN
+F 3 "~" H 3450 5100 50  0001 C CNN
+	1    3450 5100
+	0    1    1    0
+$EndComp
+Text Label 4300 5100 2    50   ~ 0
+0V5
+Text Notes 2850 5800 0    50   ~ 0
+Offset voltage
+Wire Notes Line
+	2850 4850 2850 5700
+Text Notes 2850 5950 0    50   ~ 0
+1.225 V * 1000/(1450+1000) = 0.5 V
+$Comp
+L ElectricGoKart:LM4041CFTA D4
+U 1 1 60504C24
+P 3750 5500
+F 0 "D4" V 3950 5750 50  0000 R CNN
+F 1 "LM4041CFTA" V 3850 6100 50  0000 R CNN
+F 2 "ElectricGoKart:LM4041" H 3750 5700 50  0001 C CNN
+F 3 "https://www.mouser.dk/datasheet/2/115/LM4041-10542.pdf" H 3750 5700 50  0001 C CNN
+	1    3750 5500
+	0    -1   -1   0
+$EndComp
+Wire Wire Line
+	3750 5100 3750 5200
+$Comp
+L power:GND #PWR08
+U 1 1 6050AF5E
+P 3750 5500
+F 0 "#PWR08" H 3750 5250 50  0001 C CNN
+F 1 "GND" H 3750 5350 50  0000 C CNN
+F 2 "" H 3750 5500 50  0001 C CNN
+F 3 "" H 3750 5500 50  0001 C CNN
+	1    3750 5500
+	1    0    0    -1
+$EndComp
+$Comp
+L Device:R R14
+U 1 1 6051185B
+P 4000 5100
+F 0 "R14" V 3900 5100 50  0000 C CNN
+F 1 "1.43k" V 4000 5100 50  0000 C CNN
+F 2 "Resistor_SMD:R_0603_1608Metric" V 3930 5100 50  0001 C CNN
+F 3 "~" H 4000 5100 50  0001 C CNN
+	1    4000 5100
+	0    1    1    0
+$EndComp
+Wire Wire Line
+	3750 5100 3850 5100
+Connection ~ 3750 5100
+$Comp
+L Device:R R20
+U 1 1 6051721E
+P 4300 5350
+F 0 "R20" V 4200 5350 50  0000 C CNN
+F 1 "1k" V 4300 5350 50  0000 C CNN
+F 2 "Resistor_SMD:R_0603_1608Metric" V 4230 5350 50  0001 C CNN
+F 3 "~" H 4300 5350 50  0001 C CNN
+	1    4300 5350
+	-1   0    0    1
+$EndComp
+Wire Wire Line
+	4150 5100 4300 5100
+Wire Wire Line
+	4300 5100 4300 5200
+$Comp
+L power:GND #PWR011
+U 1 1 6051D44D
+P 4300 5500
+F 0 "#PWR011" H 4300 5250 50  0001 C CNN
+F 1 "GND" H 4300 5350 50  0000 C CNN
+F 2 "" H 4300 5500 50  0001 C CNN
+F 3 "" H 4300 5500 50  0001 C CNN
+	1    4300 5500
+	1    0    0    -1
+$EndComp
+Wire Notes Line
+	4500 4850 4500 5700
+Wire Notes Line
+	4500 5700 2850 5700
+Wire Notes Line
+	2850 4850 4500 4850
+Text Notes 2900 5550 0    50   ~ 0
+1.225 V reference
+Wire Wire Line
+	3100 5100 3300 5100
+Wire Wire Line
+	3600 5100 3750 5100
+Wire Wire Line
+	4800 1550 5000 1550
+Wire Wire Line
+	4800 3600 5000 3600
 $EndSCHEMATC

Commit message: Removed some buttons and added LEDs. Finished placing the components on the PCB.
Changed lines of the file:
@@
 $EndDescr
 Text HLabel 1550 1700 0    50   Input ~ 0
+Phase2_In
+Text HLabel 1550 3750 0    50   Input ~ 0
 Phase1_In
-Text HLabel 1550 3750 0    50   Input ~ 0
-Phase2_In
 Text HLabel 5000 1550 2    50   Output ~ 0
+Phase2_ADC
+Text HLabel 5000 3600 2    50   Output ~ 0
 Phase1_ADC
-Text HLabel 5000 3600 2    50   Output ~ 0
-Phase2_ADC
 $Comp
 L Device:R R4
@@
 	1000 4600 1000 2750
 Text Notes 1000 2650 0    50   ~ 0
+Phase 2 current measurement
+Text Notes 1000 4700 0    50   ~ 0
 Phase 1 current measurement
-Text Notes 1000 4700 0    50   ~ 0
-Phase 2 current measurement
 Wire Wire Line
 	2100 4950 2100 5050
