File: PCBs/Interfaceboard/Currents.sch (KiCad schematic (older format))
At the start: 0 parts

Commit message: Merge of 'Analog Board' into main (#2)
* Added analog board schematics and finished PCB.
* Added a few documentation files.
Parts:
- added C1, C10, C5, C6: 100n, Capacitor_SMD:C_0603_1608Metric, symbol Device:C
- added C11, C13: 10µ, Capacitor_SMD:C_0805_2012Metric, symbol Device:C
- added C2, C4, C7, C9: 100p, Capacitor_SMD:C_0603_1608Metric, symbol Device:C
- added C3, C8: 1n, Capacitor_SMD:C_0603_1608Metric, symbol Device:C
- added D1, D2: 5 V, Diode_SMD:D_SOD-523, symbol Device:D_TVS
- added D4: LM4041CFTA, ElectricGoKart:LM4041, symbol ElectricGoKart:LM4041CFTA
- added FB1, FB2: 400 mA, 1k5, Inductor_SMD:L_0805_2012Metric, symbol Device:Ferrite_Bead_Small
- added R1, R3, R7, R9: 20k, Resistor_SMD:R_0603_1608Metric, symbol Device:R
- added R10, R4: 56, Resistor_SMD:R_1210_3225Metric, symbol Device:R
- added R11, R5: 3.09, Resistor_SMD:R_0603_1608Metric, symbol Device:R
- added R12, R6: DNP, Resistor_SMD:R_0603_1608Metric, symbol Device:R
- added R13: 5.1k, Resistor_SMD:R_0603_1608Metric, symbol Device:R
- added R14: 1.43k, Resistor_SMD:R_0603_1608Metric, symbol Device:R
- added R2, R8: 54.9, Resistor_SMD:R_1210_3225Metric, symbol Device:R
- added R20: 1k, Resistor_SMD:R_0603_1608Metric, symbol Device:R
- added U1, U2: AD8420ARMZ, ElectricGoKart:AD8420ARMZ, symbol ElectricGoKart:AD8420ARMZ
Connections:
- net labels added: +15V, +15V_Filt, +3V3_Ref, -15V, -15V_Filt, 0V5, GND, Phase1_ADC, Phase1_In, Phase2_ADC, Phase2_In
- wire segments 0 -> 129
Other:
- note added: "1.225 V * 1000/(1450+1000) = 0.5 V"
- note added: "1.225 V reference"
- note added: "Caps 5%"
- note added: "Offset voltage"
- note added: "P = 0.08 W"
- note added: "P = 0.73 W"
- note added: "Phase 1 current measurement"
- note added: "Phase 2 current measurement"
- note added: "Power supply stabilization"
- note added: "RFI Filter:\nf_c,diff = 1/(2*pi*R*(2*C_common+C_ground)) = 3789 Hz\nf_c,comm = 1/(2*pi*R*C_ground) = 79577 Hz\n\nDifferential phase delay at 333 Hz:\n-arctan(2*pi*333*R*(2*C_common+C_ground)) = -5 degrees"
- note added: "Tolerance =<1%"
