File: PCBs/Interfaceboard/Misc.sch (KiCad schematic (older format))
At the start: 8 parts, among them SW1 PTS645

Commit message: Removed some buttons and added LEDs. Finished placing the components on the PCB.
Parts:
- R?: renamed from R21; footprint Resistor_SMD:R_0603_1608Metric -> (none)
- R?: renamed from R22; footprint Resistor_SMD:R_0603_1608Metric -> (none)
- renumbered D5 to D?, D6 to D?
Changed lines of the file:
@@
 	1950 3850 2150 3850
 $Comp
-L Device:R R21
+L Device:R R?
 U 1 1 6051770E
 P 2250 2200
-F 0 "R21" V 2150 2200 50  0000 C CNN
+F 0 "R?" V 2150 2200 50  0000 C CNN
 F 1 "270" V 2250 2200 50  0000 C CNN
-F 2 "Resistor_SMD:R_0603_1608Metric" V 2180 2200 50  0001 C CNN
+F 2 "" V 2180 2200 50  0001 C CNN
 F 3 "~" H 2250 2200 50  0001 C CNN
 	1    2250 2200
@@
 $EndComp
 $Comp
-L Device:R R22
+L Device:R R?
 U 1 1 60517EA4
 P 2250 2650
-F 0 "R22" V 2150 2650 50  0000 C CNN
+F 0 "R?" V 2150 2650 50  0000 C CNN
 F 1 "270" V 2250 2650 50  0000 C CNN
-F 2 "Resistor_SMD:R_0603_1608Metric" V 2180 2650 50  0001 C CNN
+F 2 "" V 2180 2650 50  0001 C CNN
 F 3 "~" H 2250 2650 50  0001 C CNN
 	1    2250 2650
@@
 	1950 2650 2100 2650
 $Comp
-L Device:LED D5
+L Device:LED D?
 U 1 1 6051A708
 P 2650 2200
-F 0 "D5" H 2643 1945 50  0000 C CNN
+F 0 "D?" H 2643 1945 50  0000 C CNN
 F 1 "150060SS75000" H 2643 2036 50  0000 C CNN
 F 2 "LED_SMD:LED_0603_1608Metric" H 2650 2200 50  0001 C CNN
@@
 $EndComp
 $Comp
-L Device:LED D6
+L Device:LED D?
 U 1 1 6051AED5
 P 2650 2650
-F 0 "D6" H 2643 2395 50  0000 C CNN
+F 0 "D?" H 2643 2395 50  0000 C CNN
 F 1 "150060VS75000" H 2643 2486 50  0000 C CNN
 F 2 "LED_SMD:LED_0603_1608Metric" H 2650 2650 50  0001 C CNN
@@
 	2400 2650 2500 2650
 $Comp
-L power:GND #PWR0106
+L power:GND #PWR?
 U 1 1 6051B7BE
 P 3050 2800
-F 0 "#PWR0106" H 3050 2550 50  0001 C CNN
+F 0 "#PWR?" H 3050 2550 50  0001 C CNN
 F 1 "GND" H 3055 2627 50  0000 C CNN
 F 2 "" H 3050 2800 50  0001 C CNN
