File: PCBs/Inverterboard/dc_link/dc_link.kicad_pcb (KiCad board)
At the start: 2 copper layers, 200 x 71.9 mm, 55 parts

Commit message: Made final Gerber files for all boards.
Routing:
- net +BATT: track 126.6 -> 7.10 mm
Other:
- board text added: "DC-Link Board Spring 2021 Group 1 University of Southern Denmark"
